File: Hardware/Kicad/Port1.kicad_sch (KiCad schematic)
At the start: 81 parts, among them IC22 LT5560, IC23 THS4521IDGKR, IC24 ADL5801, IC25 NCP702-1.8, IC26 MCP33131D-10-E/MS, J2 SMA, T1 B012-617DB-1-63-B331

Commit message: some tests
Changed lines of the file:
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@@
 (kicad_sch
-	(version 20231120)
+	(version 20250114)
 	(generator "eeschema")
-	(generator_version "8.0")
+	(generator_version "9.0")
 	(paper "A3")
 	(title_block
@@
 		(company "LibreVNA")
 	)
+	(text "Downconverter to 1.IF (ca. 250kHz)"
+		(exclude_from_sim no)
+		(at 78.74 271.78 0)
+		(effects
+			(font
+				(size 1.778 1.5113)
+			)
+			(justify left bottom)
+		)
+	)
+	(text "(28 Ohm impedance)"
+		(exclude_from_sim no)
+		(at 314.96 30.48 0)
+		(effects
+			(font
+				(size 1.778 1.5113)
+			)
+			(justify left bottom)
+		)
+	)
+	(text "-3db pad"
+		(exclude_from_sim no)
+		(at 63.5 27.94 0)
+		(effects
+			(font
+				(size 1.778 1.5113)
+			)
+			(justify left bottom)
+		)
+	)
+	(text "Cut wire if \nattenuator placed"
+		(exclude_from_sim no)
+		(at 93.218 74.676 90)
+		(effects
+			(font
+				(size 1.27 1.0795)
+			)
+			(justify left bottom)
+		)
+	)
+	(text "Return loss bridge"
+		(exclude_from_sim no)
+		(at 96.52 27.94 0)
+		(effects
+			(font
+				(size 1.778 1.5113)
+			)
+			(justify left bottom)
+		)
+	)
+	(text "Final IF amplifier and ADC driver"
+		(exclude_from_sim no)
+		(at 160.02 271.78 0)
+		(effects
+			(font
+				(size 1.778 1.5113)
+			)
+			(justify left bottom)
+		)
+	)
+	(text "P1db: 0dbm"
+		(exclude_from_sim no)
+		(at 95.504 247.396 0)
+		(effects
+			(font
+				(size 1.778 1.5113)
+			)
+			(justify left bottom)
+		)
+	)
+	(text "Downconverter to 1.IF (ca. 60MHz)"
+		(exclude_from_sim no)
+		(at 175.514 21.336 0)
+		(effects
+			(font
+				(size 1.778 1.5113)
+			)
+			(justify left bottom)
+		)
+	)
+	(text "-10db pad"
+		(exclude_from_sim no)
+		(at 322.58 27.94 0)
+		(effects
+			(font
+				(size 1.778 1.5113)
+			)
+			(justify left bottom)
+		)
+	)
+	(text "300kHz lowpass"
+		(exclude_from_sim no)
+		(at 233.68 271.78 0)
+		(effects
+			(font
+				(size 1.778 1.5113)
+			)
+			(justify left bottom)
+		)
+	)
+	(text "60MHz lowpass and conversion from\n250 Ohm to 28 Ohm impedance"
+		(exclude_from_sim no)
+		(at 259.08 30.48 0)
+		(effects
+			(font
+				(size 1.778 1.5113)
+			)
+			(justify left bottom)
+		)
+	)
+	(text "1MS/s ADC"
+		(exclude_from_sim no)
+		(at 307.34 251.46 0)
+		(effects
+			(font
+				(size 1.778 1.5113)
+			)
+			(justify left bottom)
+		)
+	)
 	(junction
 		(at 154.94 63.5)
@@
 		)
 	)
-	(text "Downconverter to 1.IF (ca. 250kHz)"
-		(exclude_from_sim no)
-		(at 78.74 271.78 0)
-		(effects
-			(font
-				(size 1.778 1.5113)
-			)
-			(justify left bottom)
-		)
-	)
-	(text "(28 Ohm impedance)"
-		(exclude_from_sim no)
-		(at 314.96 30.48 0)
-		(effects
-			(font
-				(size 1.778 1.5113)
-			)
-			(justify left bottom)
-		)
-	)
-	(text "-3db pad"
-		(exclude_from_sim no)
-		(at 63.5 27.94 0)
-		(effects
-			(font
-				(size 1.778 1.5113)
-			)
-			(justify left bottom)
-		)
-	)
-	(text "Cut wire if \nattenuator placed"
-		(exclude_from_sim no)
-		(at 93.218 74.676 90)
-		(effects
-			(font
-				(size 1.27 1.0795)
-			)
-			(justify left bottom)
-		)
-	)
-	(text "Return loss bridge"
-		(exclude_from_sim no)
-		(at 96.52 27.94 0)
-		(effects
-			(font
-				(size 1.778 1.5113)
-			)
-			(justify left bottom)
-		)
-	)
-	(text "Final IF amplifier and ADC driver"
-		(exclude_from_sim no)
-		(at 160.02 271.78 0)
-		(effects
-			(font
-				(size 1.778 1.5113)
-			)
-			(justify left bottom)
-		)
-	)
-	(text "P1db: 0dbm"
-		(exclude_from_sim no)
-		(at 95.504 247.396 0)
-		(effects
-			(font
-				(size 1.778 1.5113)
-			)
-			(justify left bottom)
-		)
-	)
-	(text "Downconverter to 1.IF (ca. 60MHz)"
-		(exclude_from_sim no)
-		(at 175.514 21.336 0)
-		(effects
-			(font
-				(size 1.778 1.5113)
-			)
-			(justify left bottom)
-		)
-	)
-	(text "-10db pad"
-		(exclude_from_sim no)
-		(at 322.58 27.94 0)
-		(effects
-			(font
-				(size 1.778 1.5113)
-			)
-			(justify left bottom)
-		)
-	)
-	(text "300kHz lowpass"
-		(exclude_from_sim no)
-		(at 233.68 271.78 0)
-		(effects
-			(font
-				(size 1.778 1.5113)
-			)
-			(justify left bottom)
-		)
-	)
-	(text "60MHz lowpass and conversion from\n250 Ohm to 28 Ohm impedance"
-		(exclude_from_sim no)
-		(at 259.08 30.48 0)
-		(effects
-			(font
-				(size 1.778 1.5113)
-			)
-			(justify left bottom)
-		)
-	)
-	(text "1MS/s ADC"
-		(exclude_from_sim no)
-		(at 307.34 251.46 0)
-		(effects
-			(font
-				(size 1.778 1.5113)
-			)
-			(justify left bottom)
-		)
-	)
 	(label "RF_PORT1_LO1_CR"
 		(at 186.69 33.02 0)
-		(fields_autoplaced yes)
 		(effects
 			(font
@@
 	(label "RF_PORT1_LO1_CRC"
 		(at 193.04 53.34 270)
-		(fields_autoplaced yes)
 		(effects
 			(font
@@
 	(label "RF_PORT1_LO1_C"
 		(at 167.64 33.02 0)
-		(fields_autoplaced yes)
 		(effects
 			(font
