File: Hardware/Kicad/PowerSupply.kicad_sch (KiCad schematic)
At the start: 65 parts, among them IC1 MIC2253, IC2 LM3370, IC3 LDL212PU50R, IC4 LDL212PU50R, IC5 LDL212PU50R, IC6 LDL212PU50R, J1 PJ-014D, Q1 SSM3J338R, Q2 SSM3J338R

Commit message: some tests
Connections:
- net PWR_DET is gone; now on net +5V: J1.3, Q1.1 (G), Q2.1 (G), R125.1
Other:
- moved on the sheet: Q1
Changed lines of the file:
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@@
 (kicad_sch
-	(version 20231120)
+	(version 20250114)
 	(generator "eeschema")
-	(generator_version "8.0")
+	(generator_version "9.0")
 	(paper "A3")
 	(title_block
@@
 		(company "LibreVNA")
 	)
+	(text "Port 2 Mixers, up to 200mA"
+		(exclude_from_sim no)
+		(at 368.046 132.334 0)
+		(effects
+			(font
+				(size 1.778 1.5113)
+			)
+			(justify left bottom)
+		)
+	)
+	(text "Source and 1.LO, up to 350mA"
+		(exclude_from_sim no)
+		(at 368.046 202.184 0)
+		(effects
+			(font
+				(size 1.778 1.5113)
+			)
+			(justify left bottom)
+		)
+	)
+	(text "I2C address: 0x42"
+		(exclude_from_sim no)
+		(at 215.9 190.5 0)
+		(effects
+			(font
+				(size 1.778 1.5113)
+			)
+			(justify left bottom)
+		)
+	)
+	(text "Port 1 Mixers, up to 200mA"
+		(exclude_from_sim no)
+		(at 368.046 98.044 0)
+		(effects
+			(font
+				(size 1.778 1.5113)
+			)
+			(justify left bottom)
+		)
+	)
+	(text "Reference Mixers, up to 200mA"
+		(exclude_from_sim no)
+		(at 368.046 166.624 0)
+		(effects
+			(font
+				(size 1.778 1.5113)
+			)
+			(justify left bottom)
+		)
+	)
 	(junction
 		(at 287.02 138.43)
@@
 	)
 	(junction
+		(at 68.58 60.96)
+		(diameter 0)
+		(color 0 0 0 0)
+	)
+	(junction
 		(at 110.49 104.14)
 		(diameter 0)
@@
 	(wire
 		(pts
-			(xy 82.55 50.8) (xy 88.9 50.8)
+			(xy 68.58 25.4) (xy 88.9 25.4)
 		)
 		(stroke
@@
 	(wire
 		(pts
-			(xy 57.15 50.8) (xy 72.39 50.8)
+			(xy 66.04 25.4) (xy 58.42 25.4)
 		)
 		(stroke
@@
 	(wire
 		(pts
-			(xy 77.47 58.42) (xy 77.47 60.96)
+			(xy 63.5 33.02) (xy 63.5 60.96)
 		)
 		(stroke
@@
 	(wire
 		(pts
+			(xy 66.04 25.4) (xy 66.04 50.8)
+		)
+		(stroke
+			(width 0.1524)
+			(type solid)
+		)
+	)
+	(wire
+		(pts
 			(xy 83.82 226.06) (xy 86.36 226.06)
 		)
@@
 	(wire
 		(pts
+			(xy 88.9 25.4) (xy 88.9 50.8)
+		)
+		(stroke
+			(width 0.1524)
+			(type solid)
+		)
+	)
+	(wire
+		(pts
 			(xy 355.6 96.52) (xy 355.6 104.14)
 		)
@@
 	(wire
 		(pts
+			(xy 68.58 60.96) (xy 88.9 60.96)
+		)
+		(stroke
+			(width 0.1524)
+			(type solid)
+		)
+	)
+	(wire
+		(pts
 			(xy 140.97 233.68) (xy 140.97 226.06)
 		)
@@
 	(wire
 		(pts
-			(xy 77.47 60.96) (xy 88.9 60.96)
+			(xy 63.5 60.96) (xy 68.58 60.96)
 		)
 		(stroke
@@
 	(wire
 		(pts
+			(xy 66.04 50.8) (xy 57.15 50.8)
+		)
+		(stroke
+			(width 0.1524)
+			(type solid)
+		)
+	)
+	(wire
+		(pts
 			(xy 60.96 185.42) (xy 45.72 185.42)
 		)
@@
 		)
 	)
-	(text "Port 2 Mixers, up to 200mA"
-		(exclude_from_sim no)
-		(at 368.046 132.334 0)
-		(effects
-			(font
-				(size 1.778 1.5113)
-			)
-			(justify left bottom)
-		)
-	)
-	(text "Source and 1.LO, up to 350mA"
-		(exclude_from_sim no)
-		(at 368.046 202.184 0)
-		(effects
-			(font
-				(size 1.778 1.5113)
-			)
-			(justify left bottom)
-		)
-	)
-	(text "I2C address: 0x42"
-		(exclude_from_sim no)
-		(at 215.9 190.5 0)
-		(effects
-			(font
-				(size 1.778 1.5113)
-			)
-			(justify left bottom)
-		)
-	)
-	(text "Port 1 Mixers, up to 200mA"
-		(exclude_from_sim no)
-		(at 368.046 98.044 0)
-		(effects
-			(font
-				(size 1.778 1.5113)
-			)
-			(justify left bottom)
-		)
-	)
-	(text "Reference Mixers, up to 200mA"
-		(exclude_from_sim no)
-		(at 368.046 166.624 0)
-		(effects
-			(font
-				(size 1.778 1.5113)
-			)
-			(justify left bottom)
-		)
-	)
 	(label "USB_5V"
-		(at 86.36 50.8 0)
-		(fields_autoplaced yes)
+		(at 86.36 25.4 0)
 		(effects
 			(font
@@
 	(label "VREG6V_COMP"
 		(at 110.49 132.08 0)
-		(fields_autoplaced yes)
 		(effects
 			(font
@@
 	(label "VREGINT_SW"
 		(at 118.11 185.42 0)
-		(fields_autoplaced yes)
 		(effects
 			(font
@@
 	(label "VREG3V3_SW"
 		(at 118.11 226.06 0)
-		(fields_autoplaced yes)
 		(effects
 			(font
@@
 	(label "VREG6V_FB"
 		(at 110.49 127 0)
-		(fields_autoplaced yes)
 		(effects
 			(font
@@
 	(label "VREG6V_OVP"
 		(at 110.49 121.92 0)
-		(fields_autoplaced yes)
 		(effects
 			(font
@@
 	(label "VREG6V_SW"
 		(at 101.6 104.14 0)
-		(fields_autoplaced yes)
 		(effects
 			(font
@@
 	(label "PWR_DET"
 		(at 64.77 66.04 0)
-		(fields_autoplaced yes)
 		(effects
 			(font
@@
 	(label "VREG5V{slash}4"
 		(at 328.93 208.28 0)
-		(fields_autoplaced yes)
 		(effects
 			(font
@@
 	(label "VREG5V{slash}1"
 		(at 327.66 104.14 0)
-		(fields_autoplaced yes)
 		(effects
 			(font
@@
 	(label "VREG5V{slash}2"
 		(at 327.66 138.43 0)
-		(fields_autoplaced yes)
 		(effects
 			(font
@@
 	(label "VREG5V{slash}3"
 		(at 328.93 172.72 0)
-		(fields_autoplaced yes)
 		(effects
 			(font
@@
 	(label "VREG6V_SWD"
 		(at 129.54 104.14 0)
-		(fields_autoplaced yes)
 		(effects
 			(font
@@
 	(label "VREG3V3_SWL"
 		(at 143.51 226.06 0)
-		(fields_autoplaced yes)
 		(effects
 			(font
@@
 	(label "VREG6V_SS"
 		(at 76.2 132.08 0)
-		(fields_autoplaced yes)
 		(effects
 			(font
@@
 	(symbol
 		(lib_id "Device:Q_PMOS_GSD")
-		(at 77.47 53.34 90)
+		(at 63.5 27.94 90)
 		(unit 1)
 		(exclude_from_sim no)
@@
 		(fields_autoplaced yes)
 		(property "Reference" "Q1"
-			(at 77.47 41.91 90)
+			(at 63.5 16.51 90)
 			(effects
 				(font
@@
 		)
 		(property "Value" "SSM3J338R"
-			(at 77.47 44.45 90)
+			(at 63.5 19.05 90)
 			(effects
 				(font
@@
 		)
 		(property "Footprint" "Package_TO_SOT_SMD:SOT-23"
-			(at 74.93 48.26 0)
+			(at 60.96 22.86 0)
 			(effects
 				(font
@@
 		)
 		(property "Datasheet" ""
-			(at 77.47 53.34 0)
+			(at 63.5 27.94 0)
 			(effects
 				(font
@@
 		)
 		(property "Description" ""
-			(at 77.47 53.34 0)
+			(at 63.5 27.94 0)
 			(effects
 				(font
@@
 		)
 		(property "MPN" "SSM3J338R"
-			(at 77.47 53.34 0)
+			(at 63.5 27.94 0)
 			(effects
 				(font
@@
 		)
 		(property "Characteristic" ""
-			(at 77.47 53.34 0)
+			(at 63.5 27.94 0)
 			(effects
 				(font
@@
 		)
 		(property "Comment" "PMOS"
-			(at 77.47 46.99 90)
+			(at 63.5 21.59 90)
 			(effects
 				(font
