File: Hardware/Kicad/ReferenceSignal.kicad_sch (KiCad schematic)
At the start: 70 parts, among them IC32 THS4521IDGKR, IC33 ADL5801, IC34 NCP702-1.8, IC35 MCP33131D-10-E/MS, IC36 LT5560, T3 B012-617DB-1-63-B331

Commit message: some tests
Changed lines of the file:
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@@
 (kicad_sch
-	(version 20231120)
+	(version 20250114)
 	(generator "eeschema")
-	(generator_version "8.0")
+	(generator_version "9.0")
 	(paper "A3")
 	(title_block
